File: hardware/vfd_clock_display_board/vfd_clock_display_board.kicad_sch (KiCad schematic)
At the start: 90 parts, among them J1 Conn_01x12_Pin, J2 Conn_01x02_Pin, Q1 2N3906, Q1 MMDT5551, Q11 2N3906, Q12 2N3906, Q13 2N3906, Q14 2N3906, Q15 2N3906, Q16 2N3906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

Commit message: start redesigning display board
Parts:
- added C2 (x4): 1uF, Fab:C_1206, symbol Fab:C_1206
- added J3: Conn_PinHeader_1x03_P2.54mm_Horizontal_SMD, fab:PinHeader_1x03_P2.54mm_Horizontal_SMD, symbol Fab:Conn_PinHeader_1x03_P2.54mm_Horizontal_SMD
- added J4: Conn_01x10_MountingPin, Connector_FFC-FPC:Hirose_FH12-10S-0.5SH_1x10-1MP_P0.50mm_Horizontal, symbol Connector_Generic_MountingPin:Conn_01x10_MountingPin
- added U3, U4, U5, U6: LED_ADDR_Worldsemi_WS2812B, Fab:LED_RGB_CreeLED_CLV1A-FKB, symbol Fab:LED_ADDR_Worldsemi_WS2812B
Connections:
- net PWR_3V3: now also J3.2 (Pin_2)
- net PWR_5V: now also C2.1, C2.1, C2.1, C2.1, J3.3 (Pin_3)
- net PWR_GND: now also J3.1 (Pin_1), U3.3 (VSS), U4.3 (VSS), U5.3 (VSS), U6.3 (VSS)
- new net: C2.2, U4.1 (VDD)
- new net: U4.2 (DOUT), U5.4 (DIN)
- new net: U3.2 (DOUT), U4.4 (DIN)
- new net: C2.2, U5.1 (VDD)
- new net: C2.2, U3.1 (VDD)
- new net: U5.2 (DOUT), U6.4 (DIN)
- new net: C2.2, U6.1 (VDD)
Other:
- moved on the sheet: J1, J2

Commit message: Further hardware redesign
Parts:
- removed J1: Conn_01x12_Pin, Connector_PinSocket_2.54mm:PinSocket_1x12_P2.54mm_Vertical, symbol Connector:Conn_01x12_Pin
- removed J4: Conn_01x10_MountingPin, Connector_FFC-FPC:Hirose_FH12-10S-0.5SH_1x10-1MP_P0.50mm_Horizontal, symbol Connector_Generic_MountingPin:Conn_01x10_MountingPin
- added D1 (x3): LED_1206, fab:LED_1206, symbol Fab:LED_1206
- added J1: Conn_01x10_MountingPin, Connector_FFC-FPC:Molex_200528-0100_1x10-1MP_P1.00mm_Horizontal, symbol Connector_Generic_MountingPin:Conn_01x10_MountingPin
- added R13 (x3): 5.1K, Fab:R_1206, symbol Fab:R_1206
- L1: footprint Fab:L_1210 -> Inductor_SMD:L_Changjiang_FNR6045S
Connections:
- net 27V: now also R13.1
- net OE: now also J1.1 (Pin_1)
- net PWR_3V3: now also R13.1
- net PWR_5V: now also R13.1
- net PWR_GND: now also D1.1 (K), D1.1 (K), D1.1 (K), J1.MP (MountPin)
- net RCLK: now also J1.7 (Pin_7)
- net SER_IN: now also J1.6 (Pin_6)
- net SRCLK: now also J1.5 (Pin_5)
- net TLV_EN: now also J1.2 (Pin_2)
- net VFD0_EN: now also J1.4 (Pin_4)
- net VFD1_EN: now also J1.3 (Pin_3)
- net VFD2_EN: now also J1.9 (Pin_9)
- net VFD3_EN: now also J1.8 (Pin_8)
- net LED_DIN: now reaches U3.4 (DIN)
- net LED_DIN: now also J1.10 (Pin_10)
- new net: D1.2 (A), R13.2 (x3)
Other:
- note added: "RGB LEDs"
- moved on the sheet: C2, J2, U3, U4, U5, U6
