File: hardware/vfd_clock_display_board/vfd_clock_display_board.kicad_sch (KiCad schematic)
At the start: 105 parts, among them J1 Conn_01x10_MountingPin, J2 Conn_01x02_Pin, J3 Conn_PinHeader_1x03_P2.54mm_H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, Q1 2N3906, Q1 MMDT5551, Q11 2N3906, Q12 2N3906, Q13 2N3906, Q14 2N3906, Q15 2N3906, Q16 2N3906, Q18 2N3906, Q19 2N3906, Q2 MMDT5551, Q3 2N3906, Q3 MMDT5551, Q4 MMDT5551, Q5 2N3906, Q5 MMDT5551, Q6 MMDT5551, Q7 2N3906, U1 74HC595, U2 TLV61046ADB, U3 LED_ADDR_Worldsemi_WS2812B, U4 LED_ADDR_Worldsemi_WS2812B, U5 LED_ADDR_Worldsemi_WS2812B, U6 LED_ADDR_Worldsemi_WS2812B

Commit message: Move main board code to its own folder, update display board to match latest
Parts:
- removed C2 (x4): 1uF, Fab:C_1206, symbol Fab:C_1206
- removed D1 (x3): LED_1206, fab:LED_1206, symbol Fab:LED_1206
- removed J1: Conn_01x10_MountingPin, Connector_FFC-FPC:Molex_200528-0100_1x10-1MP_P1.00mm_Horizontal, symbol Connector_Generic_MountingPin:Conn_01x10_MountingPin
- removed J3: Conn_PinHeader_1x03_P2.54mm_Horizontal_SMD, fab:PinHeader_1x03_P2.54mm_Horizontal_SMD, symbol Fab:Conn_PinHeader_1x03_P2.54mm_Horizontal_SMD
- removed R13 (x3): 5.1K, Fab:R_1206, symbol Fab:R_1206
- removed U3, U4, U5, U6: LED_ADDR_Worldsemi_WS2812B, Fab:LED_RGB_CreeLED_CLV1A-FKB, symbol Fab:LED_ADDR_Worldsemi_WS2812B
- added J1: Conn_01x12_Pin, Connector_PinSocket_2.54mm:PinSocket_1x12_P2.54mm_Vertical, symbol Connector:Conn_01x12_Pin
- L1: footprint Inductor_SMD:L_Changjiang_FNR6045S -> Fab:L_1210
- renumbered Q13 to Q10, Q7 to Q11, Q14 to Q12, Q5 to Q13, Q6 to Q14, Q18 to Q16, Q16 to Q17, Q19 to Q18, Q3 to Q2, Q1 to Q3, Q11 to Q4, Q3 to Q5, Q12 to Q6, Q2 to Q7, Q4 to Q8, Q5 to Q9, R43 to R10, R6 to R11, R44 to R12, R23 to R13, R24 to R14, R29 to R15, R30 to R16, R28 to R17, R27 to R18, R26 to R19, R25 to R20, R7 to R21, R8 to R22, R45 to R23, R46 to R24, R35 to R25, R51 to R26, R36 to R27, R37 to R28, R52 to R29, R39 to R3, R53 to R30, R38 to R31, R54 to R32, R31 to R33, R55 to R35, R56 to R36, R61 to R37, R62 to R38, R57 to R39, R40 to R4, R63 to R40, R10 to R41, R11 to R42, R32 to R43, R33 to R44, R58 to R45, R59 to R46, R64 to R47, R65 to R48, R60 to R49, R3 to R5, R66 to R50, R12 to R51, R12 to R52, R13 to R53, R13 to R54, R12 to R55, R12 to R56, R13 to R57, R13 to R58, R41 to R6, R4 to R7, R5 to R8, R42 to R9, VFD1 to VFD2, VFD1 to VFD3, VFD1 to VFD4
Connections:
- net OE: now also J1.2 (Pin_2)
- net PWR_3V3: now also J1.1 (Pin_1)
- net PWR_5V: now also J1.11 (Pin_11)
- net PWR_GND: now also J1.12 (Pin_12)
- net RCLK: now also J1.8 (Pin_8)
- net SER_IN: now also J1.7 (Pin_7)
- net SRCLK: now also J1.6 (Pin_6)
- net TLV_EN: now also J1.3 (Pin_3)
- net VFD0_EN: now also J1.5 (Pin_5)
- net VFD1_EN: now also J1.4 (Pin_4)
- net VFD2_EN: now also J1.10 (Pin_10)
- net VFD3_EN: now also J1.9 (Pin_9)
Other:
- note removed: "RGB LEDs"
- moved on the sheet: J2
